File: Hardware/Boards/IO Module/IO Module/HDMI.kicad_sch (KiCad schematic)
At the start: 0 parts

Commit message: Updated IO Module Schematics
Added Power, USB hub and USB-JTAG circuits
Other:
- company: (none) -> Drexel University
- title: (none) -> HDMI Output Connector
Changed lines of the file:
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@@
 	(generator "eeschema")
 	(generator_version "8.0")
-	(paper "A4")
+	(paper "A3")
+	(title_block
+		(title "HDMI Output Connector")
+		(date "2024-07-14")
+		(rev "1.0")
+		(company "Drexel University")
+		(comment 1 "Designed by John Hofmeyr")
+	)
 )

Commit message: Completed IO Module Schematics
Parts:
- added C112, C113: 1uF, Capacitor_SMD:C_0402_1005Metric, symbol Device:C_Small
- added C114, C115, C116, C118, C124: 10uF, Capacitor_SMD:C_0603_1608Metric, symbol Device:C_Small
- added C117, C129: 10nF, Capacitor_SMD:C_0402_1005Metric, symbol Device:C_Small
- added C119, C120, C121, C122, C123, C125, C126, C127, C128, C130, C131, C132, C133, C134, C135, C136, C137, C138, C139, C140, C141, C142: 100nF, Capacitor_SMD:C_0402_1005Metric, symbol Device:C_Small
- added D7: 1V1 FLT, LED_SMD:LED_0603_1608Metric, symbol Device:LED
- added D8: BAS516, Diode_SMD:D_SOD-523, symbol Diode:BAS516
- added J4: HDMI_A, Connector_Video:HDMI_A_Molex_208658-1001_Horizontal, symbol Connector:HDMI_A
- added R70: 3.74K, Resistor_SMD:R_0402_1005Metric, symbol Device:R_US
- added R71, R80: 10K, Resistor_SMD:R_0402_1005Metric, symbol Device:R_US
- added R72: 3.3K, Resistor_SMD:R_0402_1005Metric, symbol Device:R_US
- added R73, R74: 2.2K, Resistor_SMD:R_0402_1005Metric, symbol Device:R_US
- added R75: 0R, Resistor_SMD:R_0402_1005Metric, symbol Device:R_US
- added R76: 1M, Resistor_SMD:R_0402_1005Metric, symbol Device:R_US
- added R77, R78, R79: 100K, Resistor_SMD:R_0402_1005Metric, symbol Device:R_US
- added R81, R82: 1K, Resistor_SMD:R_0402_1005Metric, symbol Device:R_US
- added R83, R84, R85, R86: 33R, Resistor_SMD:R_0402_1005Metric, symbol Device:R_US
- added R87: 7K, Resistor_SMD:R_0402_1005Metric, symbol Device:R_US
- added R88: 27K, Resistor_SMD:R_0402_1005Metric, symbol Device:R_US
- added U19: TPS74801AWDRC, Package_SON:VSON-10-1EP_3x3mm_P0.5mm_EP1.65x2.4mm_ThermalVias, symbol Regulator_Linear:TPS74801AWDRC
- added U20: SN75DP159RGZ, Package_DFN_QFN:QFN-48-1EP_7x7mm_P0.5mm_EP5.1x5.1mm, symbol IO_Module:SN75DP159
- added U21: TXB0108DQSR, Package_SON:USON-20_2x4mm_P0.4mm, symbol Logic_LevelTranslator:TXB0108DQSR
- added U22: TXB0101DCK, Package_TO_SOT_SMD:SOT-363_SC-70-6, symbol Logic_LevelTranslator:TXB0101DCK
Connections:
- new net: R87.2, U20.22 (Vsadj)
- new net: R80.2, U21.6 (OE)
- new net: C129.1, J4.SH, R76.2
- new net: D7.2 (A), R72.2
- new net: D7.1 (K), U19.3 (PG)
- new net: D8.2 (A), R88.2
- new net: C117.1, U19.7 (SS)
- new net: J4.14 (UTILITY), R75.2
- new net +1V8: C114.1, C131.2, C141.2, R81.2, R82.2, U19.1 (IN), U19.2 (IN), U19.5 (EN), U21.16 (VCCB), U22.1 (V_{CCA})
- new net +3V3: C112.1, C124.1, C125.2, C126.2, C130.2, C142.2, R72.1, R77.2, R78.2, R88.1, U19.4 (BIAS), U20.13 (VCC), U20.43 (VCC), U21.5 (VCCA), U22.6 (V_{CCB})
- new net +5V: C113.1, J4.18 (+5V), R73.2, R74.2
- new net FPGA_I2C_SCL: R83.2
- new net FPGA_I2C_SDA: R84.2
- new net GND: C112.2, C113.2, C114.2, C115.2, C116.2, C117.2, C118.2, C119.1, C120.1, C121.1, C122.1, C123.1, C124.2, C125.1, C126.1, C129.2, C130.1, C131.1, C140.1, C141.1, C142.1, J4.11 (CKS), J4.17 (GND), J4.2 (D2S), J4.5 (D1S), J4.8 (D0S), R71.1, R75.1, R76.1, R79.1, R80.1, R87.1, U19.11 (GND), U19.6 (GND), U20.17 (NC), U20.19 (GND), U20.30 (GND), U20.41 (GND), U20.49 (EPAD), U20.7 (GND), U21.15 (GND), U22.2 (GND)
- new net HDMI_AUX_N: C138.2
- new net HDMI_AUX_P: C139.2
- new net HDMI_CEC: U22.3 (A)
- new net HDMI_CEC_EN: U21.12 (B7)
- new net HDMI_CLK_N: C136.2
- new net HDMI_CLK_P: C137.2
- new net HDMI_C_AUX_N: C138.1, U20.44 (AUX_SRCn)
- new net HDMI_C_AUX_P: C139.1, U20.45 (AUX_SRCp)
- new net HDMI_C_CEC: D8.1 (K), J4.13 (CEC), U22.4 (B)
- new net HDMI_C_CLK_N: C136.1, J4.12 (CK-), U20.12 (IN_CLKn), U20.25 (OUT_CLKn)
- new net HDMI_C_CLK_P: C137.1, J4.10 (CK+), U20.11 (IN_CLKp), U20.26 (OUT_CLKp)
- new net HDMI_C_D0_N: C134.1, J4.9 (D0-), U20.28 (OUT_D0n), U20.9 (IN_D0n)
- new net HDMI_C_D0_P: C135.1, J4.7 (D0+), U20.29 (OUT_D0p), U20.8 (IN_D0p)
- new net HDMI_C_D1_N: C132.1, J4.6 (D1-), U20.31 (OUT_D1n), U20.6 (IN_D1n)
- new net HDMI_C_D1_P: C133.1, J4.4 (D1+), U20.32 (OUT_D1p), U20.5 (IN_D1p)
- new net HDMI_C_D2_N: C127.1, J4.3 (D2-), U20.3 (IN_D2n), U20.34 (OUT_D2n)
- new net HDMI_C_D2_P: C128.1, J4.1 (D2+), U20.2 (IN_D2p), U20.35 (OUT_D2p)
- new net HDMI_C_HPD: J4.19 (HPD), U20.33 (HPD_SNK)
- new net HDMI_C_SCL: J4.15 (SCL), R73.1, U20.38 (SCL_SINK)
- new net HDMI_C_SDA: J4.16 (SDA), R74.1, U20.39 (SDA_SINK)
- new net HDMI_D0_N: C134.2
- new net HDMI_D0_P: C135.2
- new net HDMI_D1_N: C132.2
- new net HDMI_D1_P: C133.2
- new net HDMI_D2_N: C127.2
- new net HDMI_D2_P: C128.2
- new net HDMI_EQ_SEL: U21.17 (B4)
- new net HDMI_F_CEC_EN: R79.2, U20.18 (CEC_EN), U21.9 (A7), U22.5 (OE)
- new net HDMI_F_EQ_SEL: R77.1, U20.21 (EQ_SEL/A0), U21.4 (A4)
- new net HDMI_F_I2C_EN: U20.10 (I2C_EN/PIN), U21.2 (A2)
- new net HDMI_F_PRE_SEL: U20.20 (PRE_SEL), U21.3 (A3)
- new net HDMI_F_SEL: R78.1, U20.27 (~{HDMI_SEL}/A1), U21.7 (A5)
- new net HDMI_F_SLEW: U20.40 (SLEW_CTL), U21.10 (A8)
- new net HDMI_F_SWAP: U20.1 (SWAP/POL), U21.1 (A1)
- new net HDMI_F_TX_TERM: U20.36 (TX_TERM_CTL), U21.8 (A6)
- new net HDMI_HPD_SRC: U20.4 (HPD_SRC)
- new net HDMI_I2C_EN: U21.19 (B2)
- new net HDMI_OE: C140.2, U20.42 (OE)
- new net HDMI_PRE_SEL: U21.18 (B3)
- new net HDMI_SCL_CTL: R83.1, R85.1, U20.15 (SCL_CTL)
- new net HDMI_SCL_SRC: R81.1, U20.46 (SCL_SRC)
- new net HDMI_SDA_CTL: R84.1, R86.1, U20.16 (SDA_CTL)
- new net HDMI_SDA_SRC: R82.1, U20.47 (SDA_SRC)
- new net HDMI_SEL: U21.14 (B5)
- new net HDMI_SLEW_CTL: U21.11 (B8)
- new net HDMI_SWAP: U21.20 (B1)
- new net HDMI_TX_TERM_CTL: U21.13 (B6)
- new net I2C1_SCL: R85.2
- new net I2C1_SDA: R86.2
- new net PP1V1H_FB: R70.1, R71.2, U19.8 (FB)
- new net PP_1V1_HDMI: C115.1, C116.1, C118.1, C119.2, C120.2, C121.2, C122.2, C123.2, R70.2, U19.10 (OUT), U19.9 (OUT), U20.14 (VDD), U20.23 (VDD), U20.24 (VDD), U20.37 (VDD), U20.48 (VDD)
Other:
- note added: "1V1 Core LDO"
- note added: "I2C Pullups on Top Sheet"

Commit message: Updated SCH with notes & annotations
Connections:
- net HDMI_C_CLK_N: no longer J4.12 (CK-), U20.25 (OUT_CLKn)
- net HDMI_C_CLK_P: no longer J4.10 (CK+), U20.26 (OUT_CLKp)
- net HDMI_C_D0_N: no longer J4.9 (D0-), U20.28 (OUT_D0n)
- net HDMI_C_D0_P: no longer J4.7 (D0+), U20.29 (OUT_D0p)
- net HDMI_C_D1_N: no longer J4.6 (D1-), U20.31 (OUT_D1n)
- net HDMI_C_D1_P: no longer J4.4 (D1+), U20.32 (OUT_D1p)
- net HDMI_C_D2_N: no longer J4.3 (D2-), U20.34 (OUT_D2n)
- net HDMI_C_D2_P: no longer J4.1 (D2+), U20.35 (OUT_D2p)
- new net HDMI_CON_CLK_N: J4.12 (CK-), U20.25 (OUT_CLKn)
- new net HDMI_CON_CLK_P: J4.10 (CK+), U20.26 (OUT_CLKp)
- new net HDMI_CON_D0_N: J4.9 (D0-), U20.28 (OUT_D0n)
- new net HDMI_CON_D0_P: J4.7 (D0+), U20.29 (OUT_D0p)
- new net HDMI_CON_D1_N: J4.6 (D1-), U20.31 (OUT_D1n)
- new net HDMI_CON_D1_P: J4.4 (D1+), U20.32 (OUT_D1p)
- new net HDMI_CON_D2_N: J4.3 (D2-), U20.34 (OUT_D2n)
- new net HDMI_CON_D2_P: J4.1 (D2+), U20.35 (OUT_D2p)
Changed lines of the file:
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@@
+		)
+	)
+	(text_box "NOTE: FPGA IO Bank is 1V8, Must use LVL Shifter"
+		(exclude_from_sim no)
+		(at 265.43 170.815 0)
+		(size 50.165 9.525)
+		(stroke
+			(width 0)
+			(type default)
+		)
+		(fill
+			(type none)
+		)
+		(effects
+			(font
+				(size 1.905 1.905)
+				(bold yes)
+			)
+			(justify left top)
 		)
 	)
@@
 		)
 	)
-	(label "HDMI_C_D1_P"
+	(label "HDMI_CON_D1_P"
 		(at 259.08 58.42 0)
 		(fields_autoplaced yes)
@@
 		)
 	)
-	(label "HDMI_C_D0_P"
+	(label "HDMI_CON_D0_P"
 		(at 259.08 63.5 0)
 		(fields_autoplaced yes)
@@
 		)
 	)
-	(label "HDMI_C_D0_N"
+	(label "HDMI_CON_D0_N"
 		(at 259.08 66.04 0)
 		(fields_autoplaced yes)
@@
 		)
 	)
-	(label "HDMI_C_D1_N"
+	(label "HDMI_CON_D1_N"
 		(at 259.08 60.96 0)
 		(fields_autoplaced yes)
@@
 		)
 	)
-	(label "HDMI_C_D2_P"
+	(label "HDMI_CON_D2_P"
 		(at 259.08 53.34 0)
 		(fields_autoplaced yes)
@@
 		)
 	)
-	(label "HDMI_C_CLK_P"
+	(label "HDMI_CON_CLK_P"
 		(at 259.08 68.58 0)
 		(fields_autoplaced yes)
@@
 		)
 	)
-	(label "HDMI_C_D2_N"
+	(label "HDMI_CON_D2_N"
 		(at 259.08 55.88 0)
 		(fields_autoplaced yes)
@@
 		)
 	)
-	(label "HDMI_C_CLK_N"
+	(label "HDMI_CON_CLK_N"
 		(at 259.08 71.12 0)
 		(fields_autoplaced yes)

Commit message: Updated PCB routing for IO Module
Parts:
- C112, C113, C117, C119, C120, C121, C122, C123, C125, C126, C127, C128, C129, C130, C131, C132, C133, C134, C135, C136, C137, C138, C139, C140, C141, C142: footprint Capacitor_SMD:C_0402_1005Metric -> Capacitor_SMD:C_0201_0603Metric
- R70, R71, R72, R73, R74, R75, R76, R77, R78, R79, R80, R81, R82, R83, R84, R85, R86, R87, R88: footprint Resistor_SMD:R_0402_1005Metric -> Resistor_SMD:R_0201_0603Metric
Changed lines of the file:
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@@
 			)
 		)
-		(property "Footprint" "Capacitor_SMD:C_0402_1005Metric"
+		(property "Footprint" "Capacitor_SMD:C_0201_0603Metric"
 			(at 165.1 134.62 0)
 			(effects
@@
 			)
 		)
-		(property "Footprint" "Capacitor_SMD:C_0402_1005Metric"
+		(property "Footprint" "Capacitor_SMD:C_0201_0603Metric"
 			(at 165.1 128.27 0)
 			(effects
@@
 			)
 		)
-		(property "Footprint" "Capacitor_SMD:C_0402_1005Metric"
+		(property "Footprint" "Capacitor_SMD:C_0201_0603Metric"
 			(at 165.1 106.68 0)
 			(effects
@@
 			)
 		)
-		(property "Footprint" "Resistor_SMD:R_0402_1005Metric"
+		(property "Footprint" "Resistor_SMD:R_0201_0603Metric"
 			(at 256.794 152.146 90)
 			(effects
@@
 			)
 		)
-		(property "Footprint" "Capacitor_SMD:C_0402_1005Metric"
+		(property "Footprint" "Capacitor_SMD:C_0201_0603Metric"
 			(at 165.1 114.3 0)
 			(effects
@@
 			)
 		)
-		(property "Footprint" "Capacitor_SMD:C_0402_1005Metric"
+		(property "Footprint" "Capacitor_SMD:C_0201_0603Metric"
 			(at 180.34 82.55 0)
 			(effects
@@
 			)
 		)
-		(property "Footprint" "Capacitor_SMD:C_0402_1005Metric"
+		(property "Footprint" "Capacitor_SMD:C_0201_0603Metric"
 			(at 144.78 57.15 0)
 			(effects
@@
 			)
 		)
-		(property "Footprint" "Resistor_SMD:R_0402_1005Metric"
+		(property "Footprint" "Resistor_SMD:R_0201_0603Metric"
 			(at 162.814 178.816 90)
 			(effects
@@
 			)
 		)
-		(property "Footprint" "Capacitor_SMD:C_0402_1005Metric"
+		(property "Footprint" "Capacitor_SMD:C_0201_0603Metric"
 			(at 278.13 107.95 0)
 			(effects
@@
 			)
 		)
-		(property "Footprint" "Resistor_SMD:R_0402_1005Metric"
+		(property "Footprint" "Resistor_SMD:R_0201_0603Metric"
 			(at 246.634 81.026 90)
 			(effects
@@
 			)
 		)
-		(property "Footprint" "Capacitor_SMD:C_0402_1005Metric"
+		(property "Footprint" "Capacitor_SMD:C_0201_0603Metric"
 			(at 156.21 57.15 0)
 			(effects
@@
 			)
 		)
-		(property "Footprint" "Resistor_SMD:R_0402_1005Metric"
+		(property "Footprint" "Resistor_SMD:R_0201_0603Metric"
 			(at 93.726 206.756 90)
 			(effects
@@
 			)
 		)
-		(property "Footprint" "Resistor_SMD:R_0402_1005Metric"
+		(property "Footprint" "Resistor_SMD:R_0201_0603Metric"
 			(at 339.344 106.426 90)
 			(effects
@@
 			)
 		)
-		(property "Footprint" "Capacitor_SMD:C_0402_1005Metric"
+		(property "Footprint" "Capacitor_SMD:C_0201_0603Metric"
 			(at 204.47 227.33 0)
 			(effects
@@
 			)
 		)
-		(property "Footprint" "Capacitor_SMD:C_0402_1005Metric"
+		(property "Footprint" "Capacitor_SMD:C_0201_0603Metric"
 			(at 165.1 162.56 0)
 			(effects
@@
 			)
 		)
-		(property "Footprint" "Capacitor_SMD:C_0402_1005Metric"
+		(property "Footprint" "Capacitor_SMD:C_0201_0603Metric"
 			(at 154.94 214.63 0)
 			(effects
@@
 			)
 		)
-		(property "Footprint" "Resistor_SMD:R_0402_1005Metric"
+		(property "Footprint" "Resistor_SMD:R_0201_0603Metric"
 			(at 237.744 81.026 90)
 			(effects
@@
 			)
 		)
-		(property "Footprint" "Resistor_SMD:R_0402_1005Metric"
+		(property "Footprint" "Resistor_SMD:R_0201_0603Metric"
 			(at 183.134 213.106 90)
 			(effects
@@
 			)
 		)
-		(property "Footprint" "Resistor_SMD:R_0402_1005Metric"
+		(property "Footprint" "Resistor_SMD:R_0201_0603Metric"
 			(at 56.134 69.596 90)
 			(effects
@@
 			)
 		)
-		(property "Footprint" "Resistor_SMD:R_0402_1005Metric"
+		(property "Footprint" "Resistor_SMD:R_0201_0603Metric"
 			(at 247.904 117.856 90)
 			(effects
@@
 			)
 		)
-		(property "Footprint" "Resistor_SMD:R_0402_1005Metric"
+		(property "Footprint" "Resistor_SMD:R_0201_0603Metric"
 			(at 256.794 117.856 90)
 			(effects
@@
 			)
 		)
-		(property "Footprint" "Resistor_SMD:R_0402_1005Metric"
+		(property "Footprint" "Resistor_SMD:R_0201_0603Metric"
 			(at 265.176 246.126 90)
 			(effects
@@
 			)
 		)
-		(property "Footprint" "Capacitor_SMD:C_0402_1005Metric"
+		(property "Footprint" "Capacitor_SMD:C_0201_0603Metric"
 			(at 293.37 107.95 0)
 			(effects
@@
 			)
 		)
-		(property "Footprint" "Capacitor_SMD:C_0402_1005Metric"
+		(property "Footprint" "Capacitor_SMD:C_0201_0603Metric"
 			(at 350.52 106.68 0)
 			(effects
@@
 			)
 		)
-		(property "Footprint" "Resistor_SMD:R_0402_1005Metric"
+		(property "Footprint" "Resistor_SMD:R_0201_0603Metric"
 			(at 93.726 197.866 90)
 			(effects
@@
 			)
 		)
-		(property "Footprint" "Resistor_SMD:R_0402_1005Metric"
+		(property "Footprint" "Resistor_SMD:R_0201_0603Metric"
 			(at 67.564 55.626 90)
 			(effects
@@
 			)
 		)
-		(property "Footprint" "Capacitor_SMD:C_0402_1005Metric"
+		(property "Footprint" "Capacitor_SMD:C_0201_0603Metric"
 			(at 179.07 57.15 0)
 			(effects
@@
 			)
 		)
-		(property "Footprint" "Capacitor_SMD:C_0402_1005Metric"
+		(property "Footprint" "Capacitor_SMD:C_0201_0603Metric"
 			(at 165.1 148.59 0)
 			(effects
@@
 			)
 		)
-		(property "Footprint" "Capacitor_SMD:C_0402_1005Metric"
+		(property "Footprint" "Capacitor_SMD:C_0201_0603Metric"
 			(at 339.09 38.1 0)
 			(effects
@@
 			)
 		)
-		(property "Footprint" "Capacitor_SMD:C_0402_1005Metric"
+		(property "Footprint" "Capacitor_SMD:C_0201_0603Metric"
 			(at 165.1 100.33 0)
 			(effects
@@
 			)
 		)
-		(property "Footprint" "Capacitor_SMD:C_0402_1005Metric"
+		(property "Footprint" "Capacitor_SMD:C_0201_0603Metric"
 			(at 165.1 120.65 0)
 			(effects
@@
 			)
 		)
-		(property "Footprint" "Capacitor_SMD:C_0402_1005Metric"
+		(property "Footprint" "Capacitor_SMD:C_0201_0603Metric"
 			(at 31.75 52.07 0)
 			(effects
@@
 			)
 		)
-		(property "Footprint" "Capacitor_SMD:C_0402_1005Metric"
+		(property "Footprint" "Capacitor_SMD:C_0201_0603Metric"
 			(at 168.91 82.55 0)
 			(effects
@@
 			)
 		)
-		(property "Footprint" "Resistor_SMD:R_0402_1005Metric"
+		(property "Footprint" "Resistor_SMD:R_0201_0603Metric"
 			(at 272.034 152.146 90)
 			(effects
@@
 			)
 		)
-		(property "Footprint" "Resistor_SMD:R_0402_1005Metric"
+		(property "Footprint" "Resistor_SMD:R_0201_0603Metric"
 			(at 93.726 214.376 90)
 			(effects
@@
 			)
 		)
-		(property "Footprint" "Capacitor_SMD:C_0402_1005Metric"
+		(property "Footprint" "Capacitor_SMD:C_0201_0603Metric"
 			(at 33.02 26.67 0)
 			(effects
@@
 			)
 		)
-		(property "Footprint" "Capacitor_SMD:C_0402_1005Metric"
+		(property "Footprint" "Capacitor_SMD:C_0201_0603Metric"
 			(at 167.64 57.15 0)
 			(effects
@@
 			)
 		)
-		(property "Footprint" "Resistor_SMD:R_0402_1005Metric"
+		(property "Footprint" "Resistor_SMD:R_0201_0603Metric"
 			(at 93.726 190.246 90)
 			(effects
@@
 			)
 		)
-		(property "Footprint" "Resistor_SMD:R_0402_1005Metric"
+		(property "Footprint" "Resistor_SMD:R_0201_0603Metric"
 			(at 67.564 45.466 90)
 			(effects
@@
 			)
 		)
-		(property "Footprint" "Resistor_SMD:R_0402_1005Metric"
+		(property "Footprint" "Resistor_SMD:R_0201_0603Metric"
 			(at 153.924 178.816 90)
 			(effects
@@
 			)
 		)
-		(property "Footprint" "Capacitor_SMD:C_0402_1005Metric"
+		(property "Footprint" "Capacitor_SMD:C_0201_0603Metric"
 			(at 133.35 57.15 0)
 			(effects
@@
 			)
 		)
-		(property "Footprint" "Capacitor_SMD:C_0402_1005Metric"
+		(property "Footprint" "Capacitor_SMD:C_0201_0603Metric"
 			(at 165.1 142.24 0)
 			(effects
@@
 			)
 		)
-		(property "Footprint" "Capacitor_SMD:C_0402_1005Metric"
+		(property "Footprint" "Capacitor_SMD:C_0201_0603Metric"
 			(at 219.71 227.33 0)
 			(effects
@@
 			)
 		)
-		(property "Footprint" "Resistor_SMD:R_0402_1005Metric"
+		(property "Footprint" "Resistor_SMD:R_0201_0603Metric"
 			(at 322.326 106.426 90)
 			(effects
@@
 			)
 		)
-		(property "Footprint" "Capacitor_SMD:C_0402_1005Metric"
+		(property "Footprint" "Capacitor_SMD:C_0201_0603Metric"
 			(at 165.1 156.21 0)
 			(effects
