File: Hardware/Boards/IO Module/IO Module/Camera FPC.kicad_sch (KiCad schematic)
At the start: 0 parts

Commit message: Updated IO Module Schematics
Added Power, USB hub and USB-JTAG circuits
Other:
- company: (none) -> Drexel University
- title: (none) -> Camera FPC Connector
Changed lines of the file:
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@@
 	(generator "eeschema")
 	(generator_version "8.0")
-	(paper "A4")
+	(paper "A3")
+	(title_block
+		(title "Camera FPC Connector")
+		(date "2024-07-14")
+		(rev "1.0")
+		(company "Drexel University")
+		(comment 1 "Designed by John Hofmeyr")
+	)
 )

Commit message: Completed IO Module Schematics
Parts:
- added C143, C144, C145: 100nF, Capacitor_SMD:C_0402_1005Metric, symbol Device:C_Small
- added C146, C147: 10nF, Capacitor_SMD:C_0402_1005Metric, symbol Device:C_Small
- added C148: 10uF, Capacitor_SMD:C_0603_1608Metric, symbol Device:C_Small
- added J5: Cam FPC, Connector_FFC-FPC:TE_2-1734839-2_1x22-1MP_P0.5mm_Horizontal, symbol Connector_Generic_MountingPin:Conn_01x22_MountingPin
- added R100, R101, R102, R99: 33R, Resistor_SMD:R_0402_1005Metric, symbol Device:R_US
- added R89, R90: 4.7K, Resistor_SMD:R_0402_1005Metric, symbol Device:R_US
- added R91, R92, R93, R94, R95, R96, R97, R98: 10K, Resistor_SMD:R_0402_1005Metric, symbol Device:R_US
- added U23: SN65DPHY440SS, Package_DFN_QFN:QFN-28-1EP_3x6mm_P0.5mm_EP1.7x4.75mm, symbol IO_Module:SN65DPHY440SS
Connections:
- new net +1V8: C143.2, U23.11 (VCC)
- new net +3V3: C148.1, J5.22 (Pin_22)
- new net CAM_CLK_N: J5.9 (Pin_9), U23.19 (DBCN)
- new net CAM_CLK_P: J5.8 (Pin_8), U23.20 (DBCP)
- new net CAM_D0_N: J5.3 (Pin_3), U23.23 (DB0N)
- new net CAM_D0_P: J5.2 (Pin_2), U23.24 (DB0P)
- new net CAM_D1_N: J5.6 (Pin_6), U23.21 (DB1N)
- new net CAM_D1_P: J5.5 (Pin_5), U23.22 (DB1P)
- new net CAM_D2_N: J5.12 (Pin_12), U23.17 (DB2N)
- new net CAM_D2_P: J5.11 (Pin_11), U23.18 (DB2P)
- new net CAM_D3_N: J5.15 (Pin_15), U23.15 (DB3N)
- new net CAM_D3_P: J5.14 (Pin_14), U23.16 (DB3P)
- new net CAM_LED_EN: J5.18 (Pin_18)
- new net CAM_PWR_EN: J5.17 (Pin_17)
- new net CAM_SCL: J5.20 (Pin_20), R101.1, R99.1
- new net CAM_SDA: J5.21 (Pin_21), R100.1, R102.1
- new net CFG0: R92.1, R97.2, U23.27 (VSADJ_CFG0)
- new net CFG1: R93.1, R98.2, U23.26 (PRE_CFG1)
- new net EQ: R89.1, R94.2, U23.13 (EQ/SCL)
- new net ERC: R90.1, R95.2, U23.14 (ECR/SDA)
- new net FPGA_I2C_SCL: R99.2
- new net FPGA_I2C_SDA: R100.2
- new net GND: C143.1, C144.1, C145.1, C146.2, C147.2, C148.2, J5.1 (Pin_1), J5.10 (Pin_10), J5.13 (Pin_13), J5.16 (Pin_16), J5.19 (Pin_19), J5.4 (Pin_4), J5.7 (Pin_7), J5.MP (MountPin), R94.1, R95.1, R96.1, R97.1, R98.1, U23.29 (EPAD)
- new net I2C1_SCL: R101.2
- new net I2C1_SDA: R102.2
- new net MIPI_CLK_N: U23.6 (DACN)
- new net MIPI_CLK_P: U23.5 (DACP)
- new net MIPI_D0_N: U23.2 (DA0N)
- new net MIPI_D0_P: U23.1 (DA0P)
- new net MIPI_D1_N: U23.4 (DA1N)
- new net MIPI_D1_P: U23.3 (DA1P)
- new net MIPI_D2_N: U23.8 (DA2N)
- new net MIPI_D2_P: U23.7 (DA2P)
- new net MIPI_D3_N: U23.10 (DA3N)
- new net MIPI_D3_P: U23.9 (DA3P)
- new net MIPI_VCORE: C144.2, C145.2, C146.1, C147.1, R89.2, R90.2, R91.2, R92.2, R93.2, U23.12 (VREG_OUT), U23.25 (VDD)
- new net RST: R91.1, R96.2, U23.28 (RSTN)
Other:
- note added: "I2C Pullups on Top Sheet"

Commit message: Updated PCB routing for IO Module
Parts:
- C143, C144, C145, C146, C147: footprint Capacitor_SMD:C_0402_1005Metric -> Capacitor_SMD:C_0201_0603Metric
- R100, R101, R102, R89, R90, R91, R92, R93, R94, R95, R96, R97, R98, R99: footprint Resistor_SMD:R_0402_1005Metric -> Resistor_SMD:R_0201_0603Metric
Changed lines of the file:
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@@
 			)
 		)
-		(property "Footprint" "Resistor_SMD:R_0402_1005Metric"
+		(property "Footprint" "Resistor_SMD:R_0201_0603Metric"
 			(at 241.554 93.726 90)
 			(effects
@@
 			)
 		)
-		(property "Footprint" "Resistor_SMD:R_0402_1005Metric"
+		(property "Footprint" "Resistor_SMD:R_0201_0603Metric"
 			(at 250.444 78.486 90)
 			(effects
@@
 			)
 		)
-		(property "Footprint" "Resistor_SMD:R_0402_1005Metric"
+		(property "Footprint" "Resistor_SMD:R_0201_0603Metric"
 			(at 201.676 178.816 90)
 			(effects
@@
 			)
 		)
-		(property "Footprint" "Capacitor_SMD:C_0402_1005Metric"
+		(property "Footprint" "Capacitor_SMD:C_0201_0603Metric"
 			(at 165.1 101.6 0)
 			(effects
@@
 			)
 		)
-		(property "Footprint" "Resistor_SMD:R_0402_1005Metric"
+		(property "Footprint" "Resistor_SMD:R_0201_0603Metric"
 			(at 241.554 78.486 90)
 			(effects
@@
 			)
 		)
-		(property "Footprint" "Resistor_SMD:R_0402_1005Metric"
+		(property "Footprint" "Resistor_SMD:R_0201_0603Metric"
 			(at 201.676 154.686 90)
 			(effects
@@
 			)
 		)
-		(property "Footprint" "Resistor_SMD:R_0402_1005Metric"
+		(property "Footprint" "Resistor_SMD:R_0201_0603Metric"
 			(at 201.676 162.306 90)
 			(effects
@@
 			)
 		)
-		(property "Footprint" "Capacitor_SMD:C_0402_1005Metric"
+		(property "Footprint" "Capacitor_SMD:C_0201_0603Metric"
 			(at 176.53 101.6 0)
 			(effects
@@
 			)
 		)
-		(property "Footprint" "Resistor_SMD:R_0402_1005Metric"
+		(property "Footprint" "Resistor_SMD:R_0201_0603Metric"
 			(at 268.224 93.726 90)
 			(effects
@@
 			)
 		)
-		(property "Footprint" "Resistor_SMD:R_0402_1005Metric"
+		(property "Footprint" "Resistor_SMD:R_0201_0603Metric"
 			(at 201.676 171.196 90)
 			(effects
@@
 			)
 		)
-		(property "Footprint" "Capacitor_SMD:C_0402_1005Metric"
+		(property "Footprint" "Capacitor_SMD:C_0201_0603Metric"
 			(at 153.67 101.6 0)
 			(effects
@@
 			)
 		)
-		(property "Footprint" "Resistor_SMD:R_0402_1005Metric"
+		(property "Footprint" "Resistor_SMD:R_0201_0603Metric"
 			(at 259.334 78.486 90)
 			(effects
@@
 			)
 		)
-		(property "Footprint" "Resistor_SMD:R_0402_1005Metric"
+		(property "Footprint" "Resistor_SMD:R_0201_0603Metric"
 			(at 268.224 78.486 90)
 			(effects
@@
 			)
 		)
-		(property "Footprint" "Capacitor_SMD:C_0402_1005Metric"
+		(property "Footprint" "Capacitor_SMD:C_0201_0603Metric"
 			(at 177.8 88.9 0)
 			(effects
@@
 			)
 		)
-		(property "Footprint" "Resistor_SMD:R_0402_1005Metric"
+		(property "Footprint" "Resistor_SMD:R_0201_0603Metric"
 			(at 232.664 78.486 90)
 			(effects
@@
 			)
 		)
-		(property "Footprint" "Resistor_SMD:R_0402_1005Metric"
+		(property "Footprint" "Resistor_SMD:R_0201_0603Metric"
 			(at 232.664 93.726 90)
 			(effects
@@
 			)
 		)
-		(property "Footprint" "Resistor_SMD:R_0402_1005Metric"
+		(property "Footprint" "Resistor_SMD:R_0201_0603Metric"
 			(at 259.334 93.726 90)
 			(effects
@@
 			)
 		)
-		(property "Footprint" "Resistor_SMD:R_0402_1005Metric"
+		(property "Footprint" "Resistor_SMD:R_0201_0603Metric"
 			(at 250.444 93.726 90)
 			(effects
@@
 			)
 		)
-		(property "Footprint" "Capacitor_SMD:C_0402_1005Metric"
+		(property "Footprint" "Capacitor_SMD:C_0201_0603Metric"
 			(at 142.24 101.6 0)
 			(effects
