File: Hardware/Boards/IO Module/IO Module/USB Hub.kicad_sch (KiCad schematic)
At the start: 76 parts, among them U16 TPS74801AWDRC, U18 TUSB8041, U24 TUSB1142, Y4 24Mhz

Commit message: Updates to sch
Parts:
- R54: value 33K -> 10K
- R56: value 1K -> 33K
Connections:
- net PP_VUSB is gone; now on net +1V8: R54.2
Changed lines of the file:
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@@
 	(wire
 		(pts
-			(xy 186.69 133.35) (xy 195.58 133.35)
-		)
-		(stroke
-			(width 0)
-			(type default)
-		)
-	)
-	(wire
-		(pts
 			(xy 43.18 132.08) (xy 43.18 133.35)
 		)
@@
 		)
 	)
+	(text_box "NOTE: 1V8 used since VBUS can vary from 5V to 15V\nDivider outputs ~1.3V"
+		(exclude_from_sim no)
+		(at 174.625 136.525 0)
+		(size 17.78 15.24)
+		(stroke
+			(width 0)
+			(type default)
+		)
+		(fill
+			(type none)
+		)
+		(effects
+			(font
+				(size 1.27 1.27)
+			)
+			(justify left top)
+		)
+	)
 	(text "USB Conditioning + MUX"
 		(exclude_from_sim no)
@@
 		)
 	)
-	(hierarchical_label "PP_VUSB"
-		(shape input)
-		(at 186.69 133.35 180)
-		(fields_autoplaced yes)
-		(effects
-			(font
-				(size 1.27 1.27)
-			)
-			(justify right)
-		)
-	)
 	(hierarchical_label "USB_FIFO_TX_N"
 		(shape input)
@@
 			)
 		)
-		(property "Value" "1K"
+		(property "Value" "33K"
 			(at 200.025 147.32 0)
 			(effects
@@
 			)
 		)
-		(property "Value" "33K"
+		(property "Value" "10K"
 			(at 200.025 137.16 0)
 			(effects
@@
 					(unit 1)
 				)
+			)
+		)
+	)
+	(symbol
+		(lib_id "power:+1V8")
+		(at 195.58 133.35 0)
+		(unit 1)
+		(exclude_from_sim no)
+		(in_bom yes)
+		(on_board yes)
+		(dnp no)
+		(property "Reference" "#PWR0173"
+			(at 195.58 137.16 0)
+			(effects
+				(font
+					(size 1.27 1.27)
+				)
+				(hide yes)
+			)
+		)
+		(property "Value" "+1V8"
+			(at 195.58 129.54 0)
+			(effects
+				(font
+					(size 1.27 1.27)
+				)
+			)
+		)
+		(property "Footprint" ""
+			(at 195.58 133.35 0)
+			(effects
+				(font
+					(size 1.27 1.27)
+				)
+				(hide yes)
+			)
+		)
+		(property "Datasheet" ""
+			(at 195.58 133.35 0)
+			(effects
+				(font
+					(size 1.27 1.27)
+				)
+				(hide yes)
+			)
+		)
+		(property "Description" "Power symbol creates a global label with name \"+1V8\""
+			(at 195.58 133.35 0)
+			(effects
+				(font
+					(size 1.27 1.27)
+				)
+				(hide yes)
+			)
+		)
+		(pin "1"
+		)
+		(instances
+			(project "IO Module"
+				(path "/884396b6-238b-495e-b731-e47ad2523f76/dcc99803-8acd-4632-9c0b-7f677477cf65/7fc8cead-139b-409c-a5e7-289301bfab42"
+					(reference "#PWR0173")
+					(unit 1)
+				)

Commit message: Fixed IO module firmware to read temperature correctly, added reset command to mcu
Parts:
- R104, R105, R107, R108, R109, R111, R112, R114, R115, R64, R65, R66, R69: now not fitted
Changed lines of the file:
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@@
 		(in_bom yes)
 		(on_board yes)
-		(dnp no)
+		(dnp yes)
 		(property "Reference" "R69"
 			(at 79.375 259.08 0)
@@
 		(in_bom yes)
 		(on_board yes)
-		(dnp no)
+		(dnp yes)
 		(property "Reference" "R115"
 			(at 163.195 248.92 0)
@@
 		(in_bom yes)
 		(on_board yes)
-		(dnp no)
+		(dnp yes)
 		(property "Reference" "R108"
 			(at 149.225 259.08 0)
@@
 		(in_bom yes)
 		(on_board yes)
-		(dnp no)
+		(dnp yes)
 		(property "Reference" "R64"
 			(at 65.405 259.08 0)
@@
 		(in_bom yes)
 		(on_board yes)
-		(dnp no)
+		(dnp yes)
 		(property "Reference" "R104"
 			(at 93.345 259.08 0)
@@
 		(in_bom yes)
 		(on_board yes)
-		(dnp no)
+		(dnp yes)
 		(property "Reference" "R66"
 			(at 79.375 248.92 0)
@@
 		(in_bom yes)
 		(on_board yes)
-		(dnp no)
+		(dnp yes)
 		(property "Reference" "R111"
 			(at 107.315 248.92 0)
@@
 		(in_bom yes)
 		(on_board yes)
-		(dnp no)
+		(dnp yes)
 		(property "Reference" "R107"
 			(at 135.255 259.08 0)
@@
 		(in_bom yes)
 		(on_board yes)
-		(dnp no)
+		(dnp yes)
 		(property "Reference" "R105"
 			(at 107.315 259.08 0)
@@
 		(in_bom yes)
 		(on_board yes)
-		(dnp no)
+		(dnp yes)
 		(property "Reference" "R65"
 			(at 65.405 248.92 0)
@@
 		(in_bom yes)
 		(on_board yes)
-		(dnp no)
+		(dnp yes)
 		(property "Reference" "R114"
 			(at 149.225 248.92 0)
@@
 		(in_bom yes)
 		(on_board yes)
-		(dnp no)
+		(dnp yes)
 		(property "Reference" "R112"
 			(at 121.285 248.92 0)
@@
 		(in_bom yes)
 		(on_board yes)
-		(dnp no)
+		(dnp yes)
 		(property "Reference" "R109"
 			(at 163.195 259.08 0)
