File: Hardware/Boards/FPGA Module/FPGA Module/Board_to_Boards.kicad_sch (KiCad schematic)
At the start: 2 parts, among them J1 LSHM-130-XX.X-XXX-DV-A-S-K-XX, J2 LSHM-130-XX.X-XXX-DV-A-S-K-XX

Commit message: Fixed FPGA Module Routing
Reversed B2B headers and re-routed connections to FPGA
Connections:
- net CAM_LED_EN: now also J2.57; no longer J2.03
- net CAM_PWR_EN: now also J2.59; no longer J2.01
- net FIFO_BE0: now also J1.34; no longer J1.28
- net FIFO_BE1: now also J1.32; no longer J1.30
- net FIFO_CLK: now also J1.36; no longer J1.26
- net FIFO_D0: now also J1.52; no longer J1.10
- net FIFO_D1: now also J1.50; no longer J1.12
- net FIFO_D10: now also J1.41; no longer J1.19
- net FIFO_D11: now also J1.39; no longer J1.21
- net FIFO_D12: now also J1.37; no longer J1.23
- net FIFO_D13: now also J1.35; no longer J1.25
- net FIFO_D14: now also J1.33; no longer J1.27
- net FIFO_D15: now also J1.31; no longer J1.29
- net FIFO_D2: now also J1.48; no longer J1.14
- net FIFO_D3: now also J1.46; no longer J1.16
- net FIFO_D4: now also J1.44; no longer J1.18
- net FIFO_D5: now also J1.42; no longer J1.20
- net FIFO_D6: now also J1.40; no longer J1.22
- net FIFO_D7: now also J1.38; no longer J1.24
- net FIFO_D8: now also J1.45; no longer J1.15
- net FIFO_D9: now also J1.43; no longer J1.17
- net FPGA_I2C_SCL: now also J1.01; no longer J1.59
- net FPGA_I2C_SDA: now also J1.03; no longer J1.57
- net FT600_OE: now also J2.33; no longer J2.27
- net FT600_RD: now also J1.49; no longer J1.11
- net FT600_RST: now also J2.35; no longer J2.25
- net FT600_RXE: now also J2.31; no longer J2.29
- net FT600_TXE: now also J2.29; no longer J2.31
- net FT600_WAKEUP: now also J2.37; no longer J2.23
- net FT600_WR: now also J1.51; no longer J1.09
- net GND: now also J1.11, J1.27, J1.29, J1.30, J1.47, J1.53, J1.54, J1.56, J2.01, J2.02, J2.04, J2.08, J2.14, J2.20, J2.26, J2.27, J2.32, J2.38, J2.39, J2.41, J2.43, J2.44, J2.45, J2.47, J2.49, J2.50, J2.51, J2.53, J2.55; no longer J1.06, J1.07, J1.08, J1.13, J1.31, J1.32, J1.33, J1.49, J2.05, J2.07, J2.09, J2.11, J2.12, J2.13, J2.15, J2.17, J2.18, J2.19, J2.21, J2.24, J2.30, J2.33, J2.36, J2.42, J2.48, J2.54, J2.58, J2.59, J2.60
- net HDMI_CEC: now also J2.19; no longer J2.41
- net HDMI_CLK_N: now also J2.10; no longer J2.52
- net HDMI_CLK_P: now also J2.12; no longer J2.50
- net HDMI_D0_N: now also J2.16; no longer J2.46
- net HDMI_D0_P: now also J2.18; no longer J2.44
- net HDMI_D1_N: now also J2.22; no longer J2.40
- net HDMI_D1_P: now also J2.24; no longer J2.38
- net HDMI_D2_N: now also J2.28; no longer J2.34
- net HDMI_D2_P: now also J2.30; no longer J2.32
- net HDMI_EQ_SEL: now also J2.05; no longer J2.55
- net HDMI_HPD_SRC: now also J2.09; no longer J2.51
- net HDMI_I2C_EN: now also J2.03; no longer J2.57
- net HDMI_OE: now also J2.13; no longer J2.47
- net HDMI_PRE_SEL: now also J2.07; no longer J2.53
- net HDMI_SCL_SRC: now also J2.23; no longer J2.37
- net HDMI_SDA_SRC: now also J2.25; no longer J2.35
- net HDMI_SDA_SRC_EN: now also J2.21; no longer J2.39
- net HDMI_SEL: now also J2.11; no longer J2.49
- net HDMI_SLEW_CTL: now also J2.15; no longer J2.45
- net JTAG_TCK: now also J1.02; no longer J1.60
- net JTAG_TDI: now also J1.04; no longer J1.58
- net JTAG_TDO: now also J1.06; no longer J1.56
- net JTAG_TMS: now also J1.08; no longer J1.54
- net MBUS_D0: now also J1.14; no longer J1.48
- net MBUS_D1: now also J1.16; no longer J1.46
- net MBUS_D10: now also J1.17; no longer J1.43
- net MBUS_D11: now also J1.19; no longer J1.41
- net MBUS_D12: now also J1.21; no longer J1.39
- net MBUS_D13: now also J1.23; no longer J1.37
- net MBUS_D14: now also J1.25; no longer J1.35
- net MBUS_D2: now also J1.18; no longer J1.44
- net MBUS_D3: now also J1.20; no longer J1.42
- net MBUS_D4: now also J1.22; no longer J1.40
- net MBUS_D5: now also J1.24; no longer J1.38
- net MBUS_D6: now also J1.26; no longer J1.36
- net MBUS_D7: now also J1.28; no longer J1.34
- net MBUS_D8: now also J1.13; no longer J1.47
- net MBUS_D9: now also J1.15; no longer J1.45
- net MIPI_CLK_N: now also J2.48; no longer J2.14
- net MIPI_CLK_P: now also J2.46; no longer J2.16
- net MIPI_D0_N: now also J2.36; no longer J2.26
- net MIPI_D0_P: now also J2.34; no longer J2.28
- net MIPI_D1_N: now also J2.42; no longer J2.20
- net MIPI_D1_P: now also J2.40; no longer J2.22
- net MIPI_D2_N: now also J2.54; no longer J2.08
- net MIPI_D2_P: now also J2.52; no longer J2.10
- net MIPI_D3_N: now also J2.60; no longer J2.02
- net MIPI_D3_P: now also J2.58; no longer J2.04
- net PP_VUSB: now also J1.57, J1.58, J1.59, J1.60; no longer J1.01, J1.02, J1.03, J1.04
- net TPD5_EN: now also J2.17; no longer J2.43
- net UART_RX: now also J1.10; no longer J1.52
- net UART_TX: now also J1.12; no longer J1.50
- net USB_SYSMON_D_N: now also J1.09; no longer J1.51
- net USB_SYSMON_D_P: now also J1.07; no longer J1.53
Other:
- moved on the sheet: J1, J2
