File: Hardware/Boards/FPGA Module/FPGA Module/Clock Generator.kicad_sch (KiCad schematic)
At the start: 31 parts, among them U23 Si5338A-B-GMR, Y2 12Mhz

Commit message: Generated FPGA module gerbers
Parts:
- removed TP61, TP62: Test Point, FPGA Module:Test Point 0.75mm, symbol Connector:TestPoint
- TP29, TP30, TP31, TP32, TP53, TP54, TP55, TP56, TP57: footprint FPGA Module:Test Point 0.75mm -> FPGA Module:Test Point 0.5mm No Silk
Changed lines of the file:
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@@
 	)
 	(junction
-		(at 186.69 161.29)
-		(diameter 0)
-		(color 0 0 0 0)
-	)
-	(junction
 		(at 229.87 104.14)
 		(diameter 0)
@@
 	)
 	(junction
-		(at 157.48 161.29)
-		(diameter 0)
-		(color 0 0 0 0)
-	)
-	(junction
 		(at 264.16 104.14)
 		(diameter 0)
@@
 	(wire
 		(pts
-			(xy 186.69 161.29) (xy 187.96 161.29)
-		)
-		(stroke
-			(width 0)
-			(type default)
-		)
-	)
-	(wire
-		(pts
 			(xy 281.94 147.32) (xy 281.94 144.78)
 		)
@@
 	(wire
 		(pts
-			(xy 156.21 161.29) (xy 157.48 161.29)
-		)
-		(stroke
-			(width 0)
-			(type default)
-		)
-	)
-	(wire
-		(pts
 			(xy 226.06 124.46) (xy 241.3 124.46)
 		)
@@
 		)
 	)
-	(text_box "NOTE: I2C ADDR is 0x70"
+	(text_box "NOTE: I2C ADDR is 0x70, set using IN4"
 		(exclude_from_sim no)
 		(at 162.56 127.635 0)
@@
 			)
 		)
-		(property "Footprint" "FPGA Module:Test Point 0.75mm"
+		(property "Footprint" "FPGA Module:Test Point 0.5mm No Silk"
 			(at 243.84 149.86 0)
 			(effects
@@
 			)
 		)
-		(property "Footprint" "FPGA Module:Test Point 0.75mm"
+		(property "Footprint" "FPGA Module:Test Point 0.5mm No Silk"
 			(at 231.14 160.02 0)
 			(effects
@@
 			)
 		)
-		(property "Footprint" "FPGA Module:Test Point 0.75mm"
+		(property "Footprint" "FPGA Module:Test Point 0.5mm No Silk"
 			(at 179.07 123.19 0)
 			(effects
@@
 			)
 		)
-		(property "Footprint" "FPGA Module:Test Point 0.75mm"
+		(property "Footprint" "FPGA Module:Test Point 0.5mm No Silk"
 			(at 220.98 124.46 0)
 			(effects
@@
 			)
 		)
-		(property "Footprint" "FPGA Module:Test Point 0.75mm"
+		(property "Footprint" "FPGA Module:Test Point 0.5mm No Silk"
 			(at 254 147.32 0)
 			(effects
@@
 	(symbol
 		(lib_id "Connector:TestPoint")
-		(at 156.21 161.29 0)
-		(unit 1)
-		(exclude_from_sim no)
-		(in_bom yes)
-		(on_board yes)
-		(dnp no)
-		(property "Reference" "TP61"
-			(at 153.67 156.21 0)
-			(effects
-				(font
-					(size 1.27 1.27)
-				)
-				(justify left)
-			)
-		)
-		(property "Value" "Test Point"
-			(at 151.13 155.575 0)
-			(effects
-				(font
-					(size 1.27 1.27)
-				)
-				(justify left)
-				(hide yes)
-			)
-		)
-		(property "Footprint" "FPGA Module:Test Point 0.75mm"
-			(at 161.29 161.29 0)
-			(effects
-				(font
-					(size 1.27 1.27)
-				)
-				(hide yes)
-			)
-		)
-		(property "Datasheet" "~"
-			(at 161.29 161.29 0)
-			(effects
-				(font
-					(size 1.27 1.27)
-				)
-				(hide yes)
-			)
-		)
-		(property "Description" "test point"
-			(at 156.21 161.29 0)
-			(effects
-				(font
-					(size 1.27 1.27)
-				)
-				(hide yes)
-			)
-		)
-		(pin "1"
-		)
-		(instances
-			(project "FPGA Module"
-				(path "/199f10e2-d4b4-4a27-9e84-7b1ce2ae6bf0/0c296310-f788-47f0-8a3f-43c3444563e8/e820f7e1-8a3d-4d78-a9b1-ec9a846520a7"
-					(reference "TP61")
-					(unit 1)
-				)
-			)
-		)
-	)
-	(symbol
-		(lib_id "Connector:TestPoint")
 		(at 242.57 137.16 180)
 		(unit 1)
@@
 			)
 		)
-		(property "Footprint" "FPGA Module:Test Point 0.75mm"
+		(property "Footprint" "FPGA Module:Test Point 0.5mm No Silk"
 			(at 237.49 137.16 0)
 			(effects
@@
 			)
 		)
-		(property "Footprint" "FPGA Module:Test Point 0.75mm"
+		(property "Footprint" "FPGA Module:Test Point 0.5mm No Silk"
 			(at 231.14 121.92 0)
 			(effects
@@
 			)
 		)
-		(property "Footprint" "FPGA Module:Test Point 0.75mm"
+		(property "Footprint" "FPGA Module:Test Point 0.5mm No Silk"
 			(at 220.98 162.56 0)
 			(effects
@@
 	)
 	(symbol
-		(lib_id "Connector:TestPoint")
-		(at 187.96 161.29 0)
-		(unit 1)
-		(exclude_from_sim no)
-		(in_bom yes)
-		(on_board yes)
-		(dnp no)
-		(property "Reference" "TP62"
-			(at 185.42 156.21 0)
-			(effects
-				(font
-					(size 1.27 1.27)
-				)
-				(justify left)
-			)
-		)
-		(property "Value" "Test Point"
-			(at 182.88 155.575 0)
-			(effects
-				(font
-					(size 1.27 1.27)
-				)
-				(justify left)
-				(hide yes)
-			)
-		)
-		(property "Footprint" "FPGA Module:Test Point 0.75mm"
-			(at 193.04 161.29 0)
-			(effects
-				(font
-					(size 1.27 1.27)
-				)
-				(hide yes)
-			)
-		)
-		(property "Datasheet" "~"
-			(at 193.04 161.29 0)
-			(effects
-				(font
-					(size 1.27 1.27)
-				)
-				(hide yes)
-			)
-		)
-		(property "Description" "test point"
-			(at 187.96 161.29 0)
-			(effects
-				(font
-					(size 1.27 1.27)
-				)
-				(hide yes)
-			)
-		)
-		(pin "1"
-		)
-		(instances
-			(project "FPGA Module"
-				(path "/199f10e2-d4b4-4a27-9e84-7b1ce2ae6bf0/0c296310-f788-47f0-8a3f-43c3444563e8/e820f7e1-8a3d-4d78-a9b1-ec9a846520a7"
-					(reference "TP62")
-					(unit 1)
-				)
-			)
-		)
-	)
-	(symbol
 		(lib_id "power:GND")
 		(at 229.87 111.76 0)
@@
 			)
 		)
-		(property "Footprint" "FPGA Module:Test Point 0.75mm"
+		(property "Footprint" "FPGA Module:Test Point 0.5mm No Silk"
 			(at 247.65 134.62 0)
 			(effects
