File: Hardware/Boards/FPGA Module/FPGA Module/DDR4.kicad_sch (KiCad schematic)
At the start: 39 parts, among them U4 TPS74801AWDRC, U5 MT40A512M16LY-075:E

Commit message: Updated DDR4 routing
Parts:
- R45, R48: value 10K -> 4.7K
Changed lines of the file:
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@@
 			)
 		)
-		(property "Value" "10K"
+		(property "Value" "4.7K"
 			(at 176.53 189.2299 0)
 			(effects
@@
 			)
 		)
-		(property "Value" "10K"
+		(property "Value" "4.7K"
 			(at 180.34 124.4599 0)
 			(effects

Commit message: Generated FPGA module gerbers
Parts:
- TP19, TP20: footprint FPGA Module:Test Point 0.75mm -> FPGA Module:Test Point 0.5mm No Silk
Changed lines of the file:
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@@
 			)
 		)
-		(property "Footprint" "FPGA Module:Test Point 0.75mm"
+		(property "Footprint" "FPGA Module:Test Point 0.5mm No Silk"
 			(at 264.16 54.61 0)
 			(effects
@@
 			)
 		)
-		(property "Footprint" "FPGA Module:Test Point 0.75mm"
+		(property "Footprint" "FPGA Module:Test Point 0.5mm No Silk"
 			(at 339.09 39.37 0)
 			(effects
