File: Hardware/Boards/FPGA Module/FPGA Module/FPGA Config.kicad_sch (KiCad schematic)
At the start: 36 parts, among them Q10 IRLML6244, SW2 RST, U1 XCKU3P-FFVA676, U20 MT25QUxxxxxx1xW7, U21 MAX6070BAUT12V+T

Commit message: Updates to sch
Parts:
- R121: value 4.7K -> 1K
- R123, R125: now not fitted
- R124: value 4.7K -> 1K; now not fitted
Changed lines of the file:
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@@
 		(in_bom yes)
 		(on_board yes)
-		(dnp no)
+		(dnp yes)
 		(fields_autoplaced yes)
 		(property "Reference" "R124"
@@
 			)
 		)
-		(property "Value" "4.7K"
+		(property "Value" "1K"
 			(at 208.28 226.0599 0)
 			(effects
@@
 		(in_bom yes)
 		(on_board yes)
-		(dnp no)
+		(dnp yes)
 		(fields_autoplaced yes)
 		(property "Reference" "R125"
@@
 			)
 		)
-		(property "Value" "4.7K"
+		(property "Value" "1K"
 			(at 208.28 215.8999 0)
 			(effects
@@
 		(in_bom yes)
 		(on_board yes)
-		(dnp no)
+		(dnp yes)
 		(fields_autoplaced yes)
 		(property "Reference" "R123"
