File: Hardware/Boards/Rev 2 Designs/IO Module Rev2/IO Module/HDMI Transmitter.kicad_sch (KiCad schematic)
At the start: 73 parts, among them J5 HDMI_A, U19 Sii1136, U20 TPD4E02B04DQA, U21 TPS74801AWDRC, U22 TPD4E02B04DQA, U23 L78L05_SOT89

Commit message: Updated Schematics & created pixel combiner HDL
Parts:
- R143: value 100K -> 10K
Changed lines of the file:
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@@
 			)
 		)
-		(property "Value" "100K"
+		(property "Value" "10K"
 			(at 77.47 245.11 90)
 			(effects
