File: Hardware/Boards/Rev 2 Designs/IO Module Rev2/IO Module/MCU.kicad_sch (KiCad schematic)
At the start: 21 parts, among them SW1 RST, U14 W25Q16JVUXIQ TR, U15 RP2040, Y3 12Mhz

Commit message: Rev 2 IO module complete
Parts:
- added R16, R17, R4, R5: 1K, Resistor_SMD:R_0201_0603Metric, symbol Device:R_US
- TP14: renamed from TP5; footprint TestPoint:TestPoint_Pad_D1.0mm -> IO_Module:Test Point 0.5mm No Silk
- TP15: renamed from TP6; footprint TestPoint:TestPoint_Pad_D1.0mm -> IO_Module:Test Point 0.5mm No Silk
- renumbered C68 to C70, C69 to C71, C50 to C72, C75 to C73, C70 to C75, C71 to C76, C72 to C77, C73 to C78, C76 to C79, C77 to C80, C78 to C81, D5 to D8, R47 to R56, R48 to R57, U14 to U13, U15 to U14
Connections:
- net HDMI_BUFF_EN is gone; now on net MIPI_RST_R: U14.11 (GPIO8)
- net MBUS_D12 is gone; now on net MBUS_D6: U14.35 (GPIO23)
- net MBUS_D13 is gone; now on net MBUS_D0: U14.28 (GPIO17)
- net +3V3: now also R16.2, R17.2, R4.2, R5.2
- net I2C0_SCL: now also R4.1
- net I2C0_SDA: now also R5.1
- net I2C1_SCL: now also R16.1
- net I2C1_SDA: now also R17.1
- net MBUS_D0: no longer U14.27 (GPIO16)
- net MBUS_D1: now also U14.29 (GPIO18); no longer U14.18 (GPIO15)
- net MBUS_D10: now also U14.40 (GPIO28_ADC2); no longer U14.32 (GPIO21)
- net MBUS_D11: now also U14.41 (GPIO29_ADC3); no longer U14.34 (GPIO22)
- net MBUS_D2: now also U14.30 (GPIO19); no longer U14.17 (GPIO14)
- net MBUS_D3: now also U14.31 (GPIO20); no longer U14.16 (GPIO13)
- net MBUS_D4: now also U14.32 (GPIO21); no longer U14.15 (GPIO12)
- net MBUS_D5: now also U14.34 (GPIO22); no longer U14.13 (GPIO10)
- net MBUS_D6: no longer U14.14 (GPIO11)
- net MBUS_D7: now also U14.36 (GPIO24); no longer U14.29 (GPIO18)
- net MBUS_D8: now also U14.38 (GPIO26_ADC0); no longer U14.30 (GPIO19)
- net MBUS_D9: now also U14.39 (GPIO27_ADC1); no longer U14.31 (GPIO20)
- net MIPI_RST_R: no longer U14.12 (GPIO9)
- net USBPD_CAP_MIS: now also U14.13 (GPIO10); no longer U14.40 (GPIO28_ADC2)
- net USBPD_DBG_ACC: now also U14.17 (GPIO14); no longer U14.39 (GPIO27_ADC1)
- net USBPD_FLT_IN: now also U14.15 (GPIO12); no longer U14.38 (GPIO26_ADC0)
- net USBPD_PLG_EVNT: now also U14.14 (GPIO11); no longer U14.3 (GPIO1)
- net USBPD_PLG_FLIP: now also U14.16 (GPIO13); no longer U14.2 (GPIO0)
- net USBPD_SINK_EN: now also U14.12 (GPIO9); no longer U14.36 (GPIO24)
- net VUSB_ISNS_ALRT: now also U14.3 (GPIO1); no longer U14.41 (GPIO29_ADC3)
Other:
- moved on the sheet: C70, C71, C72, C73, C74, C75, C76, C77, C78, C79, C80, C81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

Commit message: Updated Schematics & created pixel combiner HDL
Parts:
- R56: MPN RC0402JR-0710KL -> (none)
Changed lines of the file:
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@@
 			)
 		)
-		(property "MPN" "RC0402JR-0710KL"
+		(property "MPN" ""
 			(at 97.79 106.68 0)
 			(effects
