File: Hardware/Boards/Rev 2 Designs/IO Module Rev2/IO Module/Power.kicad_sch (KiCad schematic)
At the start: 82 parts, among them J1 USB_C_Receptacle, Q1 IRLML6244, Q2 IRLML6244, Q3 IRLML6244, U1 TPS25730D, U17 TPD4E02B04DQA, U2 INA700AYWFR, U26 TPD4E02B04DQA, U3 TPSM33625RDNR, U4 TPD2EUSB30A, U6 TPSM33625RDNR

Commit message: Rev 2 IO module complete
Parts:
- removed D1: 3V3 PG, LED_SMD:LED_0603_1608Metric, symbol Device:LED
- removed D8: 1V8 PG, LED_SMD:LED_0603_1608Metric, symbol Device:LED
- removed Q2, Q3: IRLML6244, Package_TO_SOT_SMD:SOT-23, symbol Transistor_FET:IRLML6244
- removed R118, R119: 2.4K, Resistor_SMD:R_0201_0603Metric, symbol Device:R_US
- removed R16, R17, R4, R5: 3.3K, Resistor_SMD:R_0201_0603Metric, symbol Device:R_US
- removed R23, R82: 47K, Resistor_SMD:R_0201_0603Metric, symbol Device:R_US
- added TP25, TP26: TestPoint, IO_Module:Test Point 0.5mm No Silk, symbol Connector:TestPoint
- renumbered C6 to C10, C7 to C11, C8 to C12, C9 to C13, C10 to C14, C11 to C15, C12 to C16, C13 to C17, C14 to C18, C15 to C19, C16 to C20, C17 to C21, C18 to C22, C19 to C23, C20 to C24, C21 to C25, C22 to C26, C23 to C27, C24 to C28, C25 to C29, C26 to C30, C27 to C31, C28 to C32, C1 to C5, C2 to C6, C3 to C7, C4 to C8, C5 to C9, Q1 to Q2, R140 to R23, R29 to R25, R24 to R26, R25 to R27, R26 to R28, R27 to R30, R28 to R31, R88 to R33, R30 to R34, R31 to R35, R32 to R36, R33 to R38, TP7 to TP11, TP8 to TP12, TP9 to TP13, U17 to U5, U26 to U7
Connections:
- net +3V3: now also R25.2, R33.2
- net 1V8_PG: now also TP25.1
- net 3V3_PG: now also TP26.1
- net PP_VUSB_R: no longer R25.2, R33.2

Commit message: Updated Schematics & created pixel combiner HDL
Parts:
- R19: value 8.06 -> 8.06K
- R6: now not fitted
Changed lines of the file:
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@@
 			)
 		)
-		(property "Value" "8.06"
+		(property "Value" "8.06K"
 			(at 226.06 120.6499 0)
 			(effects
@@
 		(in_bom yes)
 		(on_board yes)
-		(dnp no)
+		(dnp yes)
 		(fields_autoplaced yes)
 		(property "Reference" "R6"
