File: Hardware/Boards/Rev 2 Designs/IO Module Rev2/IO Module/USB Hub.kicad_sch (KiCad schematic)
At the start: 97 parts, among them U16 TPS74801AWDRC, U18 TUSB8041, U24 TUSB1142, Y4 24Mhz

Commit message: Rev 2 IO module complete
Parts:
- removed R55, R57, R67, R68: 33R, Resistor_SMD:R_0201_0603Metric, symbol Device:R_US
- added R62, R64, R73, R74: 33R, Resistor_SMD:R_0201_0603Metric, symbol Device:R_US
- U15: renamed from U16; footprint Package_SON:VSON-10-1EP_3x3mm_P0.5mm_EP1.65x2.4mm_ThermalVias -> Package_SON:VSON-10-1EP_3x3mm_P0.5mm_EP1.65x2.4mm
- U16: renamed from U18; footprint Package_DFN_QFN:QFN-64-1EP_9x9mm_P0.5mm_EP6x6mm_ThermalVias -> Package_DFN_QFN:QFN-64-1EP_9x9mm_P0.5mm_EP6x6mm
- renumbered C99 to C100, C104 to C101, C94 to C102, C109 to C103, C149 to C104, C150 to C105, C151 to C106, C152 to C107, C101 to C108, C110 to C109, C111 to C110, C103 to C111, C106 to C112, C105 to C113, C102 to C114, C108 to C115, C107 to C116, C79 to C82, C84 to C83, C85 to C84, C86 to C85, C87 to C86, C88 to C87, C89 to C88, C90 to C89, C91 to C90, C92 to C91, C80 to C92, C81 to C93, C82 to C94, C83 to C95, C95 to C96, C96 to C97, C97 to C98, C98 to C99, R106 to R100, R138 to R101, R136 to R102, R65 to R103, R66 to R104, R110 to R105, R111 to R106, R139 to R107, R137 to R108, R64 to R109, R69 to R110, R104 to R111, R105 to R112, R49 to R58, R50 to R59, R54 to R60, R51 to R61, R56 to R63, R58 to R65, R52 to R66, R59 to R67, R60 to R68, R53 to R69, R61 to R70, R63 to R71, R62 to R72, R134 to R75, R135 to R76, R115 to R77, R114 to R78, R109 to R79, R108 to R80, R120 to R81, R122 to R82, R124 to R83, R126 to R84, R128 to R85, R130 to R86, R132 to R87, R121 to R88, R123 to R89, R125 to R90, R127 to R91, R129 to R92, R131 to R93, R133 to R94, R113 to R95, R112 to R96, R116 to R97, R117 to R98, R107 to R99, TP10 to TP16, TP11 to TP17, TP12 to TP18, U24 to U17
Connections:
- net USB1D_N: now also R74.2
- net USB1D_P: now also R73.2
- net USB4D_N: now also R64.2
- net USB4D_P: now also R62.2
- net USB_FIFO_D_N: now also R64.1
- net USB_FIFO_D_P: now also R62.1
- net USB_FIFO_RX_N: now also U16.30 (USB_SSRXM_DN4); no longer U16.7 (USB_SSRXM_DN1)
- net USB_FIFO_RX_P: now also U16.29 (USB_SSRXP_DN4); no longer U16.6 (USB_SSRXP_DN1)
- net USB_FIFO_TX_N: now also U16.27 (USB_SSTXM_DN4); no longer U16.4 (USB_SSTXM_DN1)
- net USB_FIFO_TX_P: now also U16.26 (USB_SSTXP_DN4); no longer U16.3 (USB_SSTXP_DN1)
- net USB_MCU_D_N: now also R74.1
- net USB_MCU_D_P: now also R73.1

Commit message: Updated Schematics & created pixel combiner HDL
Parts:
- R101, R102: now fitted
- R61: value 100K -> 10K
Changed lines of the file:
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@@
 			)
 		)
-		(property "Value" "100K"
+		(property "Value" "10K"
 			(at 78.74 78.74 90)
 			(effects
@@
 		(in_bom yes)
 		(on_board yes)
-		(dnp yes)
+		(dnp no)
 		(property "Reference" "R101"
 			(at 59.055 248.92 0)
@@
 		(in_bom yes)
 		(on_board yes)
-		(dnp yes)
+		(dnp no)
 		(property "Reference" "R102"
 			(at 85.725 248.92 0)
