File: Hardware/Boards/Rev 2 Designs/FPGA Module Rev2/FPGA Module/Board_to_Boards.kicad_sch (KiCad schematic)
At the start: 12 parts, among them J1 LSHM-130-XX.X-XXX-DV-A-S-K-XX, J2 LSHM-130-XX.X-XXX-DV-A-S-K-XX, U18 TXB0108DQSR, U19 TXB0104RUT

Commit message: Added diagrams, papers and presentations
Parts:
- C156, C157, C158, R103, U19: now fitted
