File: Hardware/Boards/Rev 2 Designs/FPGA Module Rev2/FPGA Module/FPGA Config.kicad_sch (KiCad schematic)
At the start: 36 parts, among them Q10 IRLML6244, SW2 RST, U1 XCKU3P-FFVA676, U20 MT25QUxxxxxx1xW7, U21 MAX6070BAUT12V+T

Commit message: FPGA Module Rev 2 Layout Begun
Parts:
- removed R71, R72, R74: 0R, Resistor_SMD:R_0201_0603Metric, symbol Device:R_US
- added R100, R101, R88, R89, R90, R95: 1K, Resistor_SMD:R_0201_0603Metric, symbol Device:R_US
- renumbered C119 to C111, C120 to C112, C121 to C113, C122 to C114, C123 to C115, C124 to C116, D12 to D11, Q10 to Q3, R108 to R80, R109 to R81, R110 to R82, R111 to R83, R112 to R84, R113 to R85, R114 to R86, R118 to R87, R119 to R91, R121 to R92, R122 to R93, R123 to R94, R120 to R96, R124 to R97, R125 to R98, R126 to R99, SW2 to SW3, TP50 to TP31, TP51 to TP32, U20 to U12, U21 to U13
Connections:
- net GND: now also R101.1, R89.1, R95.1
- net MODE_0: now also R100.1, R101.2
- net MODE_1: now also R90.1, R95.2
- net MODE_2: now also R88.1, R89.2
- net DONE renamed FPGA_DONE
- new net FPGA_MCU_M0: R100.2
- new net FPGA_MCU_M1: R90.2
- new net FPGA_MCU_M2: R88.2

Commit message: Added Presentation Slides
Parts:
- R100, R88, R90: value 1K -> 8.06K
- R101, R89, R95: value 1K -> 10K
Changed lines of the file:
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@@
 		)
 	)
-	(text_box "NOTE: Default Mode set by MCU to SPI Config (M[2:0] - 001)\nFor JTAG only, set Mode to M[2:0] - 101"
+	(text_box "NOTE: Default Mode set by MCU to SPI Config (M[2:0] - 001)\nFor JTAG only, set Mode to M[2:0] - 101\n\nMCU 3V3 is divided down to 1V8 using 8K & 10K divider"
 		(exclude_from_sim no)
-		(at 48.895 160.02 0)
-		(size 43.18 8.255)
+		(at 48.895 154.94 0)
+		(size 43.18 13.335)
 		(stroke
 			(width 0)
@@
 			)
 		)
-		(property "Value" "1K"
+		(property "Value" "8.06K"
 			(at 74.93 207.0099 0)
 			(effects
@@
 			)
 		)
-		(property "Value" "1K"
+		(property "Value" "10K"
 			(at 74.93 217.1699 0)
 			(effects
@@
 			)
 		)
-		(property "Value" "1K"
+		(property "Value" "8.06K"
 			(at 74.93 234.9499 0)
 			(effects
@@
 			)
 		)
-		(property "Value" "1K"
+		(property "Value" "10K"
 			(at 74.93 245.1099 0)
 			(effects
@@
 			)
 		)
-		(property "Value" "1K"
+		(property "Value" "10K"
 			(at 74.93 189.2299 0)
 			(effects
@@
 			)
 		)
-		(property "Value" "1K"
+		(property "Value" "8.06K"
 			(at 74.93 179.0699 0)
 			(effects

Commit message: Updated main to match john-dev
Parts:
- R94, R97, R98: now fitted
Changed lines of the file:
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@@
 (kicad_sch
-	(version 20231120)
+	(version 20250114)
 	(generator "eeschema")
-	(generator_version "8.0")
+	(generator_version "9.0")
 	(paper "A3")
 	(title_block
@@
 		(comment 1 "Designed by John Hofmeyr")
 	)
+	(text "1.8V CFG"
+		(exclude_from_sim no)
+		(at 171.45 42.545 0)
+		(effects
+			(font
+				(size 3.81 3.81)
+				(thickness 2.54)
+				(bold yes)
+				(color 255 2 2 1)
+			)
+		)
+	)
+	(text_box "NOTE: Default Mode set by MCU to SPI Config (M[2:0] - 001)\nFor JTAG only, set Mode to M[2:0] - 101\n\nMCU 3V3 is divided down to 1V8 using 8K & 10K divider"
+		(exclude_from_sim no)
+		(at 48.895 154.94 0)
+		(size 43.18 13.335)
+		(margins 0.9525 0.9525 0.9525 0.9525)
+		(stroke
+			(width 0)
+			(type default)
+		)
+		(fill
+			(type none)
+		)
+		(effects
+			(font
+				(size 1.27 1.27)
+			)
+			(justify left top)
+		)
+	)
 	(junction
 		(at 92.71 96.52)
@@
 		)
 	)
-	(text_box "NOTE: Default Mode set by MCU to SPI Config (M[2:0] - 001)\nFor JTAG only, set Mode to M[2:0] - 101\n\nMCU 3V3 is divided down to 1V8 using 8K & 10K divider"
-		(exclude_from_sim no)
-		(at 48.895 154.94 0)
-		(size 43.18 13.335)
-		(stroke
-			(width 0)
-			(type default)
-		)
-		(fill
-			(type none)
-		)
-		(effects
-			(font
-				(size 1.27 1.27)
-			)
-			(justify left top)
-		)
-	)
-	(text "1.8V CFG"
-		(exclude_from_sim no)
-		(at 171.45 42.545 0)
-		(effects
-			(font
-				(size 3.81 3.81)
-				(thickness 2.54)
-				(bold yes)
-				(color 255 2 2 1)
-			)
-		)
-	)
 	(label "CFG_MEM_D3"
 		(at 201.93 101.6 180)
-		(fields_autoplaced yes)
 		(effects
 			(font
@@
 	(label "INIT_B_0"
 		(at 226.06 219.71 0)
-		(fields_autoplaced yes)
 		(effects
 			(font
@@
 	(label "CFG_MEM_CS"
 		(at 201.93 88.9 180)
-		(fields_autoplaced yes)
 		(effects
 			(font
@@
 	(label "CFG_MEM_D3"
 		(at 251.46 100.33 0)
-		(fields_autoplaced yes)
 		(effects
 			(font
@@
 	(label "JTAG_R_TD0"
 		(at 143.51 64.77 0)
-		(fields_autoplaced yes)
 		(effects
 			(font
@@
 	(label "CFG_MEM_D2"
 		(at 251.46 97.79 0)
-		(fields_autoplaced yes)
 		(effects
 			(font
@@
 	(label "CFG_MEM_D1"
 		(at 251.46 95.25 0)
-		(fields_autoplaced yes)
 		(effects
 			(font
@@
 	(label "GNDADC"
 		(at 187.96 110.49 0)
-		(fields_autoplaced yes)
 		(effects
 			(font
@@
 	(label "PUDC_B_0"
 		(at 142.24 82.55 0)
-		(fields_autoplaced yes)
 		(effects
 			(font
@@
 	(label "MODE_2"
 		(at 91.44 182.88 180)
-		(fields_autoplaced yes)
 		(effects
 			(font
@@
 	(label "PROGRAM_B_0"
 		(at 142.24 85.09 0)
-		(fields_autoplaced yes)
 		(effects
 			(font
@@
 	(label "MODE_1"
 		(at 91.44 210.82 180)
-		(fields_autoplaced yes)
 		(effects
 			(font
@@
 	(label "JTAG_R_TCK"
 		(at 143.51 62.23 0)
-		(fields_autoplaced yes)
 		(effects
 			(font
@@
 	(label "FPGA_DONE"
 		(at 201.93 76.2 180)
-		(fields_autoplaced yes)
 		(effects
 			(font
@@
 	(label "MODE_0"
 		(at 91.44 238.76 180)
-		(fields_autoplaced yes)
 		(effects
 			(font
@@
 	(label "JTAG_TDI"
 		(at 107.95 59.69 0)
-		(fields_autoplaced yes)
 		(effects
 			(font
@@
 	(label "CFG_MEM_CLK"
 		(at 201.93 91.44 180)
-		(fields_autoplaced yes)
 		(effects
 			(font
@@
 	(label "MODE_0"
 		(at 142.24 72.39 0)
-		(fields_autoplaced yes)
 		(effects
 			(font
@@
 	(label "GNDADC"
 		(at 203.2 69.85 0)
-		(fields_autoplaced yes)
 		(effects
 			(font
@@
 	(label "FPGA_VREF_P"
 		(at 138.43 101.6 0)
-		(fields_autoplaced yes)
 		(effects
 			(font
@@
 	(label "FPGA_MCU_M1"
 		(at 52.07 200.66 0)
-		(fields_autoplaced yes)
 		(effects
 			(font
@@
 	(label "FPGA_VREF_N"
 		(at 138.43 104.1855 0)
-		(fields_autoplaced yes)
 		(effects
 			(font
@@
 	(label "POR_OVERRIDE"
 		(at 142.24 87.63 0)
-		(fields_autoplaced yes)
 		(effects
 			(font
@@
 	(label "FPGA_MCU_M2"
 		(at 52.07 172.72 0)
-		(fields_autoplaced yes)
 		(effects
 			(font
@@
 	(label "JTAG_TMS"
 		(at 107.95 57.15 0)
-		(fields_autoplaced yes)
 		(effects
 			(font
@@
 	(label "FPGA_DONE"
 		(at 107.95 229.87 0)
-		(fields_autoplaced yes)
 		(effects
 			(font
@@
 	(label "PROGRAM_B_0"
 		(at 187.96 173.99 0)
-		(fields_autoplaced yes)
 		(effects
 			(font
@@
 	(label "FPGA_MCU_M0"
 		(at 52.07 228.6 0)
-		(fields_autoplaced yes)
 		(effects
 			(font
@@
 	(label "CFG_MEM_CS"
 		(at 251.46 87.63 0)
-		(fields_autoplaced yes)
 		(effects
 			(font
@@
 	(label "MODE_2"
 		(at 142.24 77.47 0)
-		(fields_autoplaced yes)
 		(effects
 			(font
@@
 	(label "MODE_1"
 		(at 142.24 74.93 0)
-		(fields_autoplaced yes)
 		(effects
 			(font
@@
 	(label "POR_OVERRIDE"
 		(at 270.51 219.71 0)
-		(fields_autoplaced yes)
 		(effects
 			(font
@@
 	(label "JTAG_TDO"
 		(at 107.95 64.77 0)
-		(fields_autoplaced yes)
 		(effects
 			(font
@@
 	(label "JTAG_R_TDI"
 		(at 143.51 59.69 0)
-		(fields_autoplaced yes)
 		(effects
 			(font
@@
 	(label "CFG_MEM_CLK"
 		(at 251.46 90.17 0)
-		(fields_autoplaced yes)
 		(effects
 			(font
@@
 	(label "CFG_MEM_D0"
 		(at 201.93 93.98 180)
-		(fields_autoplaced yes)
 		(effects
 			(font
@@
 	(label "CFG_MEM_D2"
 		(at 201.93 99.06 180)
-		(fields_autoplaced yes)
 		(effects
 			(font
@@
 	(label "PUDC_B_0"
 		(at 181.61 219.71 0)
-		(fields_autoplaced yes)
 		(effects
 			(font
@@
 	(label "CFG_MEM_D0"
 		(at 251.46 92.71 0)
-		(fields_autoplaced yes)
 		(effects
 			(font
@@
 	(label "INIT_B_0"
 		(at 201.93 78.74 180)
-		(fields_autoplaced yes)
 		(effects
 			(font
@@
 	(label "JTAG_R_TMS"
 		(at 143.51 57.15 0)
-		(fields_autoplaced yes)
 		(effects
 			(font
@@
 	(label "JTAG_TCK"
 		(at 107.95 62.23 0)
-		(fields_autoplaced yes)
 		(effects
 			(font
@@
 	(label "CFG_MEM_D1"
 		(at 201.93 96.52 180)
-		(fields_autoplaced yes)
 		(effects
 			(font
@@
 		(shape input)
 		(at 107.95 64.77 180)
-		(fields_autoplaced yes)
 		(effects
 			(font
@@
 		(shape input)
 		(at 107.95 57.15 180)
-		(fields_autoplaced yes)
 		(effects
 			(font
@@
 		(shape input)
 		(at 52.07 172.72 180)
-		(fields_autoplaced yes)
 		(effects
 			(font
@@
 		(shape input)
 		(at 52.07 228.6 180)
-		(fields_autoplaced yes)
 		(effects
 			(font
@@
 		(shape input)
 		(at 107.95 62.23 180)
-		(fields_autoplaced yes)
 		(effects
 			(font
@@
 		(shape input)
 		(at 107.95 59.69 180)
-		(fields_autoplaced yes)
 		(effects
 			(font
@@
 		(shape input)
 		(at 52.07 200.66 180)
-		(fields_autoplaced yes)
 		(effects
 			(font
@@
 		(in_bom yes)
 		(on_board yes)
-		(dnp yes)
+		(dnp no)
 		(fields_autoplaced yes)
 		(property "Reference" "R97"
@@
 		(in_bom yes)
 		(on_board yes)
-		(dnp yes)
+		(dnp no)
 		(fields_autoplaced yes)
 		(property "Reference" "R98"
@@
 		(in_bom yes)
 		(on_board yes)
-		(dnp yes)
+		(dnp no)
 		(fields_autoplaced yes)
 		(property "Reference" "R94"
