File: Hardware/Boards/Rev 2 Designs/FPGA Module Rev2/FPGA Module/FPGA_IO.kicad_sch (KiCad schematic)
At the start: 42 parts, among them Q1 FDG1024NZ, Q2 FDG1024NZ, SW1 RST, U1 XCKU3P-FFVA676, U2 Si511J200

Commit message: modified FPGA MIPI code to add ready output, modified IO module FW to initialize camera after fpga rdy goes high
Parts:
- D1, D2, D3, D4, Q1, Q2, R10, R11, R12, R13, R14, R16, R17, R18, R19, R20, R21, R22, R23, R3, R4, R7, R8, R9: now not fitted
- R15: now fitted
Changed lines of the file:
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@@
 		(in_bom yes)
 		(on_board yes)
-		(dnp no)
+		(dnp yes)
 		(property "Reference" "R19"
 			(at 92.71 345.44 90)
@@
 		(in_bom yes)
 		(on_board yes)
-		(dnp no)
+		(dnp yes)
 		(property "Reference" "R14"
 			(at 167.64 317.4999 0)
@@
 		(in_bom yes)
 		(on_board yes)
-		(dnp no)
+		(dnp yes)
 		(property "Reference" "R22"
 			(at 55.88 360.68 90)
@@
 		(in_bom yes)
 		(on_board yes)
-		(dnp no)
+		(dnp yes)
 		(property "Reference" "Q1"
 			(at 41.91 312.4199 0)
@@
 		(in_bom yes)
 		(on_board yes)
-		(dnp no)
+		(dnp yes)
 		(property "Reference" "R21"
 			(at 92.71 353.06 90)
@@
 		(in_bom yes)
 		(on_board yes)
-		(dnp no)
+		(dnp yes)
 		(property "Reference" "Q2"
 			(at 152.4 312.4199 0)
@@
 		(in_bom yes)
 		(on_board yes)
-		(dnp no)
+		(dnp yes)
 		(property "Reference" "R8"
 			(at 85.09 293.3699 0)
@@
 		(in_bom yes)
 		(on_board yes)
-		(dnp no)
+		(dnp yes)
 		(property "Reference" "R16"
 			(at 55.88 337.82 90)
@@
 		(in_bom yes)
 		(on_board yes)
-		(dnp no)
+		(dnp yes)
 		(property "Reference" "R23"
 			(at 92.71 360.68 90)
@@
 		(in_bom yes)
 		(on_board yes)
-		(dnp no)
+		(dnp yes)
 		(property "Reference" "R18"
 			(at 55.88 345.44 90)
@@
 		(in_bom yes)
 		(on_board yes)
-		(dnp no)
+		(dnp yes)
 		(property "Reference" "R10"
 			(at 158.75 293.3699 0)
@@
 		(in_bom yes)
 		(on_board yes)
-		(dnp no)
+		(dnp yes)
 		(property "Reference" "R12"
 			(at 93.98 317.4999 0)
@@
 		(in_bom yes)
 		(on_board yes)
-		(dnp no)
+		(dnp yes)
 		(property "Reference" "R9"
 			(at 121.92 293.3699 0)
@@
 		(in_bom yes)
 		(on_board yes)
-		(dnp no)
+		(dnp yes)
 		(property "Reference" "R7"
 			(at 48.26 293.3699 0)
@@
 		(in_bom yes)
 		(on_board yes)
-		(dnp no)
+		(dnp yes)
 		(property "Reference" "D3"
 			(at 125.73 302.26 90)
@@
 		(in_bom yes)
 		(on_board yes)
-		(dnp no)
+		(dnp yes)
 		(property "Reference" "R11"
 			(at 57.15 317.4999 0)
@@
 		(in_bom yes)
 		(on_board yes)
-		(dnp no)
+		(dnp yes)
 		(fields_autoplaced yes)
 		(property "Reference" "R4"
@@
 		(in_bom yes)
 		(on_board yes)
-		(dnp no)
+		(dnp yes)
 		(property "Reference" "R17"
 			(at 92.71 337.82 90)
@@
 		(in_bom yes)
 		(on_board yes)
-		(dnp no)
+		(dnp yes)
 		(property "Reference" "R20"
 			(at 55.88 353.06 90)
@@
 		(in_bom yes)
 		(on_board yes)
-		(dnp no)
+		(dnp yes)
 		(property "Reference" "R13"
 			(at 130.81 317.4999 0)
@@
 		(in_bom yes)
 		(on_board yes)
-		(dnp no)
+		(dnp yes)
 		(property "Reference" "D1"
 			(at 52.07 302.26 90)
@@
 		(in_bom yes)
 		(on_board yes)
-		(dnp no)
+		(dnp yes)
 		(property "Reference" "D2"
 			(at 88.9 302.26 90)
@@
 		(in_bom yes)
 		(on_board yes)
-		(dnp no)
+		(dnp yes)
 		(property "Reference" "D4"
 			(at 162.56 302.26 90)
@@
 		(in_bom yes)
 		(on_board yes)
-		(dnp no)
+		(dnp yes)
 		(fields_autoplaced yes)
 		(property "Reference" "R3"
@@
 		(in_bom yes)
 		(on_board yes)
-		(dnp yes)
+		(dnp no)
 		(fields_autoplaced yes)
 		(property "Reference" "R15"
@@
 		(in_bom yes)
 		(on_board yes)
-		(dnp no)
+		(dnp yes)
 		(property "Reference" "Q1"
 			(at 78.74 312.4199 0)
@@
 		(in_bom yes)
 		(on_board yes)
-		(dnp no)
+		(dnp yes)
 		(property "Reference" "Q2"
 			(at 115.57 312.4199 0)

Commit message: Added diagrams, papers and presentations
Parts:
- D1, D2, D3, D4, Q1, Q2, R10, R11, R12, R13, R14, R16, R17, R18, R19, R20, R21, R22, R23, R7, R8, R9: now fitted
