File: Hardware/Boards/Rev 2 Designs/FPGA Module Rev2/FPGA Module/FPGA_IO.kicad_sch (KiCad schematic)
At the start: 42 parts, among them Q1 FDG1024NZ, Q2 FDG1024NZ, SW1 RST, U1 XCKU3P-FFVA676, U2 Si511J200

Commit message: Updated main to match john-dev
Parts:
- R15: now fitted
- R3, R4: now not fitted
