File: Hardware/Boards/Rev 2 Designs/FPGA Module Rev2/FPGA Module/System_Controller.kicad_sch (KiCad schematic)
At the start: 30 parts, among them SW1 RST, U7 W25Q16JVUXIQ TR, U8 RP2040, Y1 12Mhz

Commit message: FPGA Module Rev 2 Layout Begun
Parts:
- renumbered C64 to C29, C65 to C30, C66 to C31, C67 to C32, C68 to C33, C69 to C34, C70 to C35, C71 to C36, C72 to C37, C74 to C38, C75 to C39, C76 to C40, D6 to D5, R50 to R28, R51 to R29, R52 to R30, R53 to R31, R54 to R32, R55 to R33, SW1 to SW2, TP21 to TP15, TP22 to TP16, TP23 to TP17, TP24 to TP18, TP25 to TP19, TP26 to TP20, TP27 to TP21, U7 to U3, U8 to U4
Connections:
- net FAN_PWM: now reaches U4.16 (GPIO13)
- net 0V9_EN renamed 5V0_EN
- net 0V9_ISNS_ALERT: no longer names the net of U4.36 (GPIO24)
- net LVL_SHIFT_EN: no longer names the net of U4.14 (GPIO11)
- net MCU_CLK: no longer names the net of U4.2 (GPIO0)
- net VMCU_1V1 renamed MCU_1V1
- no-connect marks 7 -> 9

Commit message: Rev 2 PCB's and Heatsink PCB's complete
Connections:
- net 0V85_EN: now also U4.11 (GPIO8); no longer U4.31 (GPIO20)
- net 0V85_ISNS_ALERT: now also U4.12 (GPIO9); no longer U4.18 (GPIO15)
- net 1V2_EN: now also U4.18 (GPIO15); no longer U4.13 (GPIO10)
- net 1V2_ISNS_ALERT: now also U4.13 (GPIO10); no longer U4.35 (GPIO23)
- net 1V8_EN: now also U4.31 (GPIO20); no longer U4.15 (GPIO12)
- net 1V8_ISNS_ALERT: now also U4.15 (GPIO12); no longer U4.11 (GPIO8)
- net 3V3_ISNS_ALERT: now also U4.17 (GPIO14); no longer U4.12 (GPIO9)
- net 5V0_EN: now also U4.35 (GPIO23); no longer U4.17 (GPIO14)

Commit message: modified FPGA MIPI code to add ready output, modified IO module FW to initialize camera after fpga rdy goes high
Parts:
- C29, C30, C31, C32, C33, C34, C35, C36, C37, C38, C39, C40, D5, R28, R29, R30, R31, R32, R33, SW2, U3, U4, Y1: now not fitted
Changed lines of the file:
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@@
 		(in_bom yes)
 		(on_board yes)
-		(dnp no)
+		(dnp yes)
 		(fields_autoplaced yes)
 		(property "Reference" "R32"
@@
 		(in_bom yes)
 		(on_board yes)
-		(dnp no)
+		(dnp yes)
 		(fields_autoplaced yes)
 		(property "Reference" "R31"
@@
 		(in_bom yes)
 		(on_board yes)
-		(dnp no)
+		(dnp yes)
 		(fields_autoplaced yes)
 		(property "Reference" "C29"
@@
 		(in_bom yes)
 		(on_board yes)
-		(dnp no)
+		(dnp yes)
 		(fields_autoplaced yes)
 		(property "Reference" "C34"
@@
 		(in_bom yes)
 		(on_board yes)
-		(dnp no)
+		(dnp yes)
 		(fields_autoplaced yes)
 		(property "Reference" "C37"
@@
 		(in_bom yes)
 		(on_board yes)
-		(dnp no)
+		(dnp yes)
 		(fields_autoplaced yes)
 		(property "Reference" "C40"
@@
 		(in_bom yes)
 		(on_board yes)
-		(dnp no)
+		(dnp yes)
 		(fields_autoplaced yes)
 		(property "Reference" "C33"
@@
 		(in_bom yes)
 		(on_board yes)
-		(dnp no)
+		(dnp yes)
 		(property "Reference" "U3"
 			(at 134.62 130.81 0)
@@
 		(in_bom yes)
 		(on_board yes)
-		(dnp no)
+		(dnp yes)
 		(fields_autoplaced yes)
 		(property "Reference" "C39"
@@
 		(in_bom yes)
 		(on_board yes)
-		(dnp no)
+		(dnp yes)
 		(fields_autoplaced yes)
 		(property "Reference" "R30"
@@
 		(in_bom yes)
 		(on_board yes)
-		(dnp no)
+		(dnp yes)
 		(fields_autoplaced yes)
 		(property "Reference" "U4"
@@
 		(in_bom yes)
 		(on_board yes)
-		(dnp no)
+		(dnp yes)
 		(fields_autoplaced yes)
 		(property "Reference" "C30"
@@
 		(in_bom yes)
 		(on_board yes)
-		(dnp no)
+		(dnp yes)
 		(fields_autoplaced yes)
 		(property "Reference" "R33"
@@
 		(in_bom yes)
 		(on_board yes)
-		(dnp no)
+		(dnp yes)
 		(fields_autoplaced yes)
 		(property "Reference" "C36"
@@
 		(in_bom yes)
 		(on_board yes)
-		(dnp no)
+		(dnp yes)
 		(fields_autoplaced yes)
 		(property "Reference" "C35"
@@
 		(in_bom yes)
 		(on_board yes)
-		(dnp no)
+		(dnp yes)
 		(property "Reference" "Y1"
 			(at 130.81 160.02 0)
@@
 		(in_bom yes)
 		(on_board yes)
-		(dnp no)
+		(dnp yes)
 		(property "Reference" "D5"
 			(at 290.83 177.165 0)
@@
 		(in_bom yes)
 		(on_board yes)
-		(dnp no)
+		(dnp yes)
 		(fields_autoplaced yes)
 		(property "Reference" "SW2"
@@
 		(in_bom yes)
 		(on_board yes)
-		(dnp no)
+		(dnp yes)
 		(property "Reference" "R28"
 			(at 130.81 114.3 90)
@@
 		(in_bom yes)
 		(on_board yes)
-		(dnp no)
+		(dnp yes)
 		(property "Reference" "R29"
 			(at 281.94 183.515 90)
@@
 		(in_bom yes)
 		(on_board yes)
-		(dnp no)
+		(dnp yes)
 		(fields_autoplaced yes)
 		(property "Reference" "C38"
@@
 		(in_bom yes)
 		(on_board yes)
-		(dnp no)
+		(dnp yes)
 		(fields_autoplaced yes)
 		(property "Reference" "C31"
@@
 		(in_bom yes)
 		(on_board yes)
-		(dnp no)
+		(dnp yes)
 		(fields_autoplaced yes)
 		(property "Reference" "C32"

Commit message: Added diagrams, papers and presentations
Parts:
- C29, C30, C31, C32, C33, C34, C35, C36, C37, C38, C39, C40, D5, R28, R29, R30, R31, R32, R33, SW2, U3, U4, Y1: now fitted
